Commit message: converted_2Wheel_robot_to_4WheelRobot

File: install/my_robot_description/share/my_robot_description/urdf/mobile_base.xacro (robot description, xacro)
@@ -1,4 +1,5 @@
 <?xml version="1.0"?>
 <robot xmlns:xacro="http://www.ros.org/wiki/xacro">
+    <!-- Properties -->
     <xacro:property name="base_length" value="0.6" />
     <xacro:property name="base_width" value="0.4" />
@@ -6,5 +7,7 @@
     <xacro:property name="wheel_radius" value="0.1" />
     <xacro:property name="wheel_length" value="0.05" />
+    <!-- Base footprint -->
     <link name="base_footprint" />
+    <!-- Base link -->
     <link name="base_link">
         <visual>
@@ -24,4 +27,5 @@
                            xyz="0 0 ${base_height / 2.0}" rpy="0 0 0" />
     </link>
+    <!-- Macro for a wheel -->
     <xacro:macro name="wheel_link" params="prefix">
         <link name="${prefix}_wheel_link">
@@ -43,23 +47,10 @@
         </link>
     </xacro:macro>
-    <xacro:wheel_link prefix="right" />
-    <xacro:wheel_link prefix="left" />
-    <link name="caster_wheel_link">
-        <visual>
-            <geometry>
-                <sphere radius="${wheel_radius / 2.0}" />
-            </geometry>
-            <origin xyz="0 0 0" rpy="0 0 0" />
-            <material name="grey" />
-        </visual>
-        <collision>
-            <geometry>
-                <sphere radius="${wheel_radius / 2.0}" />
-            </geometry>
-            <origin xyz="0 0 0" rpy="0 0 0" />
-        </collision>
-        <xacro:sphere_inertia m="0.5" r="${2*wheel_radius / 2.0}"
-                              xyz="0 0 0" rpy="0 0 0" />
-    </link>
+    <!-- 4 Wheels -->
+    <xacro:wheel_link prefix="rear_right" />
+    <xacro:wheel_link prefix="rear_left" />
+    <xacro:wheel_link prefix="front_right" />
+    <xacro:wheel_link prefix="front_left" />
+    <!-- Joints -->
     <joint name="base_joint" type="fixed">
         <parent link="base_footprint" />
@@ -67,20 +58,31 @@
         <origin xyz="0 0 ${wheel_radius}" rpy="0 0 0"/>
     </joint>
-    <joint name="base_right_wheel_joint" type="continuous">
+    <!-- Front Wheels (controlled directly) -->
+    <joint name="base_front_right_wheel_joint" type="continuous">
         <parent link="base_link" />
-        <child link="right_wheel_link" />
-        <origin xyz="${-base_length / 4.0} ${-(base_width + wheel_length) / 2.0} 0" rpy="0 0 0" />
+        <child link="front_right_wheel_link" />
+        <origin xyz="${base_length / 2.5} ${-(base_width + wheel_length) / 2.0} 0" rpy="0 0 0" />
         <axis xyz="0 1 0" />
     </joint>
-    <joint name="base_left_wheel_joint" type="continuous">
+    <joint name="base_front_left_wheel_joint" type="continuous">
         <parent link="base_link" />
-        <child link="left_wheel_link" />
-        <origin xyz="${-base_length / 4.0} ${(base_width + wheel_length) / 2.0} 0" rpy="0 0 0" />
+        <child link="front_left_wheel_link" />
+        <origin xyz="${base_length / 2.5} ${(base_width + wheel_length) / 2.0} 0" rpy="0 0 0" />
         <axis xyz="0 1 0" />
     </joint>
-    <joint name="base_caster_wheel_joint" type="fixed">
+    <!-- Rear Wheels (MIMIC joints) -->
+    <joint name="base_rear_right_wheel_joint" type="continuous">
         <parent link="base_link" />
-        <child link="caster_wheel_link" />
-        <origin xyz="${base_length / 3.0} 0 ${-wheel_radius / 2.0}" rpy="0 0 0" />
+        <child link="rear_right_wheel_link" />
+        <origin xyz="${-base_length / 2.5} ${-(base_width + wheel_length) / 2.0} 0" rpy="0 0 0" />
+        <axis xyz="0 1 0" />
+        <mimic joint="base_front_right_wheel_joint" multiplier="1.0" />
+    </joint>
+    <joint name="base_rear_left_wheel_joint" type="continuous">
+        <parent link="base_link" />
+        <child link="rear_left_wheel_link" />
+        <origin xyz="${-base_length / 2.5} ${(base_width + wheel_length) / 2.0} 0" rpy="0 0 0" />
+        <axis xyz="0 1 0" />
+        <mimic joint="base_front_left_wheel_joint" multiplier="1.0" />
     </joint>
 </robot>

File: install/my_robot_description/share/my_robot_description/urdf/mobile_base_gazebo.xacro (robot description, xacro)
@@ -1,29 +1,31 @@
 <?xml version="1.0"?>
 <robot xmlns:xacro="http://www.ros.org/wiki/xacro">
+    <!-- Set material colors in Gazebo -->
     <gazebo reference="base_link">
         <material>Gazebo/Blue</material>
     </gazebo>
-    <gazebo reference="right_wheel_link">
+    <gazebo reference="rear_right_wheel_link">
         <material>Gazebo/Grey</material>
     </gazebo>
-    <gazebo reference="left_wheel_link">
+    <gazebo reference="rear_left_wheel_link">
         <material>Gazebo/Grey</material>
     </gazebo>
-    <gazebo reference="caster_wheel_link">
+    <gazebo reference="front_right_wheel_link">
         <material>Gazebo/Grey</material>
-        <mu1 value="0.1" />
-        <mu2 value="0.1" />
     </gazebo>
+    <gazebo reference="front_left_wheel_link">
+        <material>Gazebo/Grey</material>
+    </gazebo>
+    <!-- Diff Drive Controller Plugin -->
     <gazebo>
         <plugin name="diff_drive_controller" filename="libgazebo_ros_diff_drive.so">
-            <!-- Update rate in Hz -->
             <update_rate>50</update_rate>
-            <!-- wheels -->
-            <left_joint>base_left_wheel_joint</left_joint>
-            <right_joint>base_right_wheel_joint</right_joint>
-            <!-- kinematics -->
-            <wheel_separation>0.45</wheel_separation>
-            <wheel_diameter>0.2</wheel_diameter>
-            <!-- output -->
+            <!-- Define LEFT and RIGHT wheel joints properly -->
+            <left_joint>base_front_left_wheel_joint</left_joint>
+            <right_joint>base_front_right_wheel_joint</right_joint>
+            <!-- Kinematics settings -->
+            <wheel_separation>0.45</wheel_separation> <!-- Distance between left and right wheels -->
+            <wheel_diameter>0.2</wheel_diameter>       <!-- Diameter of wheels -->
+            <!-- Odometry and TF -->
             <publish_odom>true</publish_odom>
             <publish_odom_tf>true</publish_odom_tf>
