Commit message: converted 2_joint arm to 6DOF

File: install/my_robot_description/share/my_robot_description/urdf/arm.xacro (robot description, xacro)
@@ -1,77 +1,115 @@
 <?xml version="1.0"?>
-<robot xmlns:xacro="http://www.ros.org/wiki/xacro">
-    <xacro:property name="arm_base_length" value="0.1" />
-    <xacro:property name="arm_base_width" value="0.1" />
-    <xacro:property name="arm_base_height" value="0.02" />
-    <xacro:property name="forearm_radius" value="0.02" />
-    <xacro:property name="forearm_length" value="0.3" />
-    <xacro:property name="hand_radius" value="0.02" />
-    <xacro:property name="hand_length" value="0.3" />
-    <link name="arm_base_link">
-        <visual>
-            <geometry>
-                <box size="${arm_base_length} ${arm_base_width} ${arm_base_height}" />
-            </geometry>
-            <origin xyz="0 0 ${arm_base_height / 2.0}" rpy="0 0 0" />
-            <material name="orange" />
-        </visual>
-        <collision>
-            <geometry>
-                <box size="${arm_base_length} ${arm_base_width} ${arm_base_height}" />
-            </geometry>
-            <origin xyz="0 0 ${arm_base_height / 2.0}" rpy="0 0 0" />
-        </collision>
-        <xacro:box_inertia m="0.5" l="${2*arm_base_length}" w="${2*arm_base_width}" h="${2*arm_base_height}"
-                           xyz="0 0 ${arm_base_height / 2.0}" rpy="0 0 0" />
+<robot xmlns:xacro="http://www.ros.org/wiki/xacro" name="my_robot_description">
+  <!-- Properties -->
+  <xacro:property name="base_radius" value="0.05"/>
+  <xacro:property name="base_height" value="0.05"/>
+  <xacro:property name="joint_radius" value="0.04"/>
+  <xacro:property name="joint_length" value="0.2"/>
+  <xacro:property name="finger_length" value="0.05"/>
+  <xacro:property name="finger_width" value="0.01"/>
+  <xacro:property name="gripper_spacing" value="0.03"/>
+  <!-- Arm Base Link -->
+  <link name="arm_base_link">
+    <visual>
+      <geometry>
+        <cylinder radius="${base_radius}" length="${base_height}"/>
+      </geometry>
+      <origin xyz="0 0 ${base_height / 2.0}" rpy="0 0 0"/>
+      <material name="blue"/>
+    </visual>
+  </link>
+  <!-- First joint connects to arm_base_link -->
+  <link name="joint_0_link">
+    <visual>
+      <geometry>
+        <cylinder radius="${joint_radius}" length="${joint_length}"/>
+      </geometry>
+      <origin xyz="0 0 ${joint_length / 2.0}" rpy="0 0 0"/>
+      <material name="grey"/>
+    </visual>
+  </link>
+  <joint name="joint_0_joint" type="revolute">
+    <parent link="arm_base_link"/>
+    <child link="joint_0_link"/>
+    <origin xyz="0 0 ${base_height}" rpy="0 0 0"/>
+    <axis xyz="0 0 1"/>
+    <limit lower="-1.57" upper="1.57" effort="100" velocity="1.0"/>
+    <dynamics friction="0.1" damping="0.1"/>
+  </joint>
+  <!-- Arm Segments -->
+  <xacro:macro name="arm_segment" params="index">
+    <link name="joint_${index}_link">
+      <visual>
+        <geometry>
+          <cylinder radius="${joint_radius}" length="${joint_length}"/>
+        </geometry>
+        <origin xyz="0 0 ${joint_length / 2.0}" rpy="0 0 0"/>
+        <material name="grey"/>
+      </visual>
     </link>
-    <link name="forearm_link">
-        <visual>
-            <geometry>
-                <cylinder radius="${forearm_radius}" length="${forearm_length}" />
-            </geometry>
-            <origin xyz="0 0 ${forearm_length / 2.0}" rpy="0 0 0" />
-            <material name="yellow" />
-        </visual>
-        <collision>
-            <geometry>
-                <cylinder radius="${forearm_radius}" length="${forearm_length}" />
-            </geometry>
-            <origin xyz="0 0 ${forearm_length / 2.0}" rpy="0 0 0" />
-        </collision>
-        <xacro:cylinder_inertia m="0.3" r="${2*forearm_radius}" h="${2*forearm_length}"
-                                xyz="0 0 ${forearm_length / 2.0}" rpy="0 0 0" />
-    </link>
-    <link name="hand_link">
-        <visual>
-            <geometry>
-                <cylinder radius="${hand_radius}" length="${hand_length}" />
-            </geometry>
-            <origin xyz="0 0 ${hand_length / 2.0}" rpy="0 0 0" />
-            <material name="orange" />
-        </visual>
-        <collision>
-             <geometry>
-                <cylinder radius="${hand_radius}" length="${hand_length}" />
-            </geometry>
-            <origin xyz="0 0 ${hand_length / 2.0}" rpy="0 0 0" />
-        </collision>
-        <xacro:cylinder_inertia m="0.3" r="${2*hand_radius}" h="${2*hand_length}"
-                                xyz="0 0 ${hand_length / 2.0}" rpy="0 0 0" />
-    </link>
-    <joint name="arm_base_forearm_joint" type="revolute">
-        <parent link="arm_base_link" />
-        <child link="forearm_link" />
-        <origin xyz="0 0 ${arm_base_height}" rpy="0 0 0" />
-        <axis xyz="0 1 0" />
-        <limit lower="0" upper="${pi/2}" effort="100" velocity="100" />
-        <dynamics friction="0.05" damping="0.1" />
+    <joint name="joint_${index}_joint" type="revolute">
+      <parent link="joint_${index - 1}_link"/>
+      <child link="joint_${index}_link"/>
+      <origin xyz="0 0 ${joint_length}" rpy="0 0 0"/>
+      <axis xyz="0 1 0"/>
+      <limit lower="-1.57" upper="1.57" effort="100" velocity="1.0"/>
+      <dynamics friction="0.1" damping="0.1"/>
     </joint>
-    <joint name="forearm_hand_joint" type="revolute">
-        <parent link="forearm_link" />
-        <child link="hand_link" />
-        <origin xyz="0 0 ${forearm_length}" rpy="0 0 0" />
-        <axis xyz="0 1 0" />
-        <limit lower="0" upper="${pi/2}" effort="100" velocity="100" />
-        <dynamics friction="0.05" damping="0.1" />
-    </joint>
+  </xacro:macro>
+  <xacro:arm_segment index="1"/>
+  <xacro:arm_segment index="2"/>
+  <xacro:arm_segment index="3"/>
+  <xacro:arm_segment index="4"/>
+  <xacro:arm_segment index="5"/>
+  <!-- Gripper Base Link -->
+  <link name="gripper_base_link">
+    <visual>
+      <geometry>
+        <box size="0.04 0.04 0.02"/>
+      </geometry>
+      <origin xyz="0 0 0.01" rpy="0 0 0"/>
+      <material name="dark_grey"/>
+    </visual>
+  </link>
+  <joint name="gripper_base_joint" type="fixed">
+    <parent link="joint_5_link"/>
+    <child link="gripper_base_link"/>
+    <origin xyz="0 0 ${joint_length}" rpy="0 0 0"/>
+  </joint>
+  <!-- Left Finger -->
+  <link name="left_finger_link">
+    <visual>
+      <geometry>
+        <box size="${finger_width} 0.02 ${finger_length}"/>
+      </geometry>
+      <origin xyz="0 0 ${finger_length / 2.0}" rpy="0 0 0"/>
+      <material name="silver"/>
+    </visual>
+  </link>
+  <joint name="left_finger_joint" type="revolute">
+    <parent link="gripper_base_link"/>
+    <child link="left_finger_link"/>
+    <origin xyz="${gripper_spacing / 2.0} 0 0.01" rpy="0 0 0"/>
+    <axis xyz="1 0 0"/>
+    <limit lower="0.0" upper="0.03" effort="10" velocity="1.0"/>
+    <dynamics friction="0.01" damping="0.01"/>
+  </joint>
+  <!-- Right Finger -->
+  <link name="right_finger_link">
+    <visual>
+      <geometry>
+        <box size="${finger_width} 0.02 ${finger_length}"/>
+      </geometry>
+      <origin xyz="0 0 ${finger_length / 2.0}" rpy="0 0 0"/>
+      <material name="silver"/>
+    </visual>
+  </link>
+  <joint name="right_finger_joint" type="revolute">
+    <parent link="gripper_base_link"/>
+    <child link="right_finger_link"/>
+    <origin xyz="-${gripper_spacing / 2.0} 0 0.01" rpy="0 0 0"/>
+    <axis xyz="1 0 0"/>
+    <limit lower="-0.03" upper="0.0" effort="10" velocity="1.0"/>
+    <dynamics friction="0.01" damping="0.01"/>
+  </joint>
 </robot>

File: install/my_robot_description/share/my_robot_description/urdf/my_robot.urdf.xacro (robot description, xacro)
@@ -5,5 +5,5 @@
     <xacro:include filename="mobile_base_gazebo.xacro" />
     <xacro:include filename="arm.xacro" />
-    <xacro:include filename="arm_gazebo.xacro" />
+    <xacro:include filename="arm1_gazebo.xacro" />
     <joint name="mobile_base_arm_joint" type="fixed">
         <parent link="base_link" />
